Commit message: committed mobile robot(not yet done)

File: urdf/mobile_robot.urdf (robot description, URDF)
Before this commit: robot mobile, 2 links, 1 joints
Links:
- added link wheel_1_link; visual cylinder length=0.05 radius=0.05
- added link wheel_2_link; visual cylinder length=0.05 radius=0.05
- added link wheel_3_link; visual cylinder length=0.05 radius=0.05
- link base_link: geometry visual box size=0.35 0.25 0.05
Joints:
- removed joint world_to_base
- added joint base_to_wheel_1: type continuous, parent base_link, child wheel_1_link, origin xyz=0.125 0.150 0.0 rpy=1.57 0 0, axis 0 0 1
- added joint base_to_wheel_2: type continuous, parent base_link, child wheel_2_link, origin xyz=-0.125 -0.150 0.0 rpy=1.57 0 0, axis 0 0 1
- added joint base_to_wheel_3: type continuous, parent base_link, child wheel_3_link, origin xyz=0 0 0.0 rpy=1.57 0 0, axis 0 0 1
- added joint base_to_world: type fixed, parent world, child base_link, origin xyz=0 0 0.05

Commit message: Complete geometry, no physics yet

File: urdf/mobile_robot.urdf (robot description, URDF)
Before this commit: robot mobile, 5 links, 4 joints
Links:
- added link wheel_4_link; visual cylinder length=0.05 radius=0.05
Joints:
- added joint base_to_wheel_4: type continuous, parent base_link, child wheel_4_link, origin xyz=0.125 -0.150 0.0 rpy=1.57 0 0, axis 0 0 1
- joint base_to_wheel_3: origin xyz=0 0 0.0 rpy=1.57 0 0 -> xyz=-0.125 0.15 0 rpy=1.57 0 0
