Commit message: added a camera link

File: urdf/mobile_robot.xacro (robot description, xacro)
@@ -56,4 +56,5 @@
         <origin rpy = "1.57 0 0" xyz = "0.125 0.150 0.0"/>
         <axis xyz = "0 0 1"/>
+        <dynamics damping="1.0" friction="1.0"/>
     </joint>
     <!--rear right wheel-->
@@ -85,4 +86,5 @@
         <origin rpy = "1.57 0 0" xyz = "-0.125 -0.150 0.0"/>
         <axis xyz = "0 0 1"/>
+        <dynamics damping="1.0" friction="1.0"/>
     </joint>
     <!--front right wheel-->
@@ -114,4 +116,5 @@
         <origin rpy = "1.57 0 0" xyz = "-0.125 0.15 0"/>
         <axis xyz = "0 0 1"/>
+        <dynamics damping="1.0" friction="1.0"/>
     </joint>
     <!--rear left wheel-->
@@ -143,4 +146,37 @@
         <origin rpy = "1.57 0 0" xyz = "0.125 -0.150 0.0"/>
         <axis xyz = "0 0 1"/>
+        <dynamics damping="1.0" friction="1.0"/>
+    </joint>
+    <!--camera-->
+    <link name="camera_link">
+    <visual>
+        <origin xyz="0 0 0" rpy="0 0 0"/>
+        <geometry>
+            <box size="0.02 0.02 0.02"/>
+        </geometry>
+        <material name="Cyan1">
+        <color rgba="0 0.9 0.9 1.0"/>
+        </material>
+    </visual>
+    <collision>
+        <origin xyz="0 0 0" rpy="0 0 0"/>
+        <geometry>
+        <box size="0.5 0.5 0.3"/>
+    </geometry>
+    </collision>
+    <inertial>
+        <origin xyz="0 0 0" rpy="0 0 0"/>
+            <mass value="0.5"/>
+        <inertia
+        ixx="0.1" ixy="0.0" ixz="0.0"
+        iyy="0.1" iyz="0.0"
+        izz="0.1"/>
+    </inertial>
+    </link>
+    <joint name="camera_to_base" type="fixed">
+        <limit effort="1000.0" lower="-3.14" upper="3.14" velocity="0.5"/>
+        <origin rpy="0 0 0" xyz="0.175 0 0"/>
+        <parent link="base_link"/>
+        <child link="camera_link"/>
     </joint>
     <!--base to world-->
@@ -148,5 +184,5 @@
         <parent link="world"/>
         <child link="base_link"/>
-        <origin xyz = "0 0 0.05"/>
+        <origin xyz = "0 0 0.5"/>
     </joint>
 </robot>

Commit message: removed world link

File: urdf/mobile_robot.xacro (robot description, xacro)
@@ -2,5 +2,4 @@
 <robot name="mobile" xmlns:xacro="http://www.ros.org/wiki/xacro">
     <xacro:include filename="$(find two_links)/urdf/mobile_gazebo.gazebo"/>
-    <link name="world"></link>
     <link name="base_link">
     <visual>
@@ -180,9 +179,3 @@
         <child link="camera_link"/>
     </joint>
-    <!--base to world-->
-    <joint name="base_to_world" type="fixed">
-        <parent link="world"/>
-        <child link="base_link"/>
-        <origin xyz = "0 0 0.5"/>
-    </joint>
 </robot>

Commit message: fixed camera collision

File: urdf/mobile_robot.xacro (robot description, xacro)
@@ -161,5 +161,5 @@
         <origin xyz="0 0 0" rpy="0 0 0"/>
         <geometry>
-        <box size="0.5 0.5 0.3"/>
+        <box size="0.02 0.02 0.02"/>
     </geometry>
     </collision>
